File: pcb/Lyra-HS.kicad_sch (KiCad schematic)
At the start: 96 parts, among them J1 Computer/Power, J2 AVR-ISP-6, SW1 SW_Push, SW19 SW_Push, SW2 SW_Push, SW20 SW_Push, SW21 SW_Push, SW22 SW_Push, SW23 SW_Push, SW24 SW_Push, SW25 SW_Push, SW3 SW_Push, SW37 SW_Push, SW38 SW_Push, SW39 SW_Push, SW4 SW_Push, SW40 SW_Push, SW41 SW_Push, SW42 SW_Push, SW43 SW_Push, SW5 SW_Push, SW55 SW_Push, SW56 SW_Push, SW57 SW_Push, SW58 SW_Push, SW59 SW_Push, SW6 SW_Push, SW60 SW_Push, SW61 SW_Push, SW7 SW_Push, SW73 SW_Push, SW74 SW_Push, SW75 SW_Push, SW76 SW_Push, SW77 SW_Push, SW78 SW_Push, SW79 SW_Push, U1 ATmega32U4-MU, U2 SRV05-4, Y1 16mhz

Commit message: Initial matrix layout
Parts:
- C1, C2, C3, C4, C5, C6: footprint Keebio:C_0402 -> Keeb.io:C_0402
- J3: renamed from J?; footprint (none) -> Lily58:TRRS_JACK_MJ4PP9
- SW1, SW19, SW2, SW20, SW21, SW22, SW23, SW24, SW25, SW3, SW37, SW38, SW39, SW4, SW40, SW41, SW42, SW43, SW5, SW55, SW56, SW57, SW58, SW59, SW6, SW60, SW61, SW7, SW73, SW74, SW75, SW76, SW77, SW78: footprint keebiocustom:MX-Alps-Choc-1U-NoLED -> Lily58:MX_Choc_Hotswap
- SW79: footprint keebiocustom:MX-Alps-Choc-2U-StabFlip-NoLED -> Lily58:MX_Choc_Hotswap
Connections:
- net DI+: now also U2.4 (IO3)
- no-connect marks 6 -> 17

Commit message: Matrix impedance optimisations
+change to desolder-friendly trrs jack footprint
Parts:
- J3: footprint Lily58:TRRS_JACK_MJ4PP9 -> Keeb.io:TRRS-PJ-320A-Dual-Overlayed; symbol Connector:AudioJack3 -> Connector:AudioJack4
- SWRST1: footprint Keebio:SW_SPST_TL3342 -> Keeb.io:SW_SPST_TL3342
- Y1: footprint Crystal:Resonator_SMD_muRata_CSTxExxV-3Pin_3.0x1.1mm_HandSoldering -> Crystal:Resonator_SMD_Murata_CSTxExxV-3Pin_3.0x1.1mm
Connections:
- net GND: now also J3.3; no longer J3.R
- net Serial: now also J3.2; no longer J3.S
- net VCC: now also J3.4; no longer J3.T
Changed lines of the file:
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@@
     )
   )
-  (global_label "Serial" (shape input) (at 101.6 110.49 0) (fields_autoplaced)
+  (global_label "Serial" (shape input) (at 110.49 115.57 0) (fields_autoplaced)
     (effects (font (size 1.27 1.27)) (justify left))
-    (property "Intersheet References" "${INTERSHEET_REFS}" (id 0) (at 109.4275 110.4106 0)
+    (property "Intersheet References" "${INTERSHEET_REFS}" (id 0) (at 118.3175 115.4906 0)
       (effects (font (size 1.27 1.27)) (justify left) hide)
     )
@@
       (effects (font (size 1.27 1.27)) (justify left))
     )
-    (property "Footprint" "Crystal:Resonator_SMD_muRata_CSTxExxV-3Pin_3.0x1.1mm_HandSoldering" (id 2) (at 190.5 53.975 0)
+    (property "Footprint" "Crystal:Resonator_SMD_Murata_CSTxExxV-3Pin_3.0x1.1mm" (id 2) (at 190.5 53.975 0)
       (effects (font (size 1.27 1.27)) hide)
     )
@@
     (property "Reference" "SWRST1" (id 0) (at 210.439 35.56 0))
     (property "Value" "SW_Push" (id 1) (at 208.1276 35.56 0))
-    (property "Footprint" "Keebio:SW_SPST_TL3342" (id 2) (at 208.28 35.56 0)
+    (property "Footprint" "Keeb.io:SW_SPST_TL3342" (id 2) (at 208.28 35.56 0)
       (effects (font (size 1.27 1.27)) hide)
     )
@@
     (pin "1")
   )
-  (symbol (lib_id "power:VCC") (at 101.6 115.57 270) (unit 1)
+  (symbol (lib_id "power:VCC") (at 110.49 110.49 270) (unit 1)
     (in_bom yes) (on_board yes) (fields_autoplaced)
-    (property "Reference" "#PWR04" (id 0) (at 97.79 115.57 0)
+    (property "Reference" "#PWR04" (id 0) (at 106.68 110.49 0)
       (effects (font (size 1.27 1.27)) hide)
     )
-    (property "Value" "VCC" (id 1) (at 105.41 115.5699 90)
+    (property "Value" "VCC" (id 1) (at 114.3 110.4899 90)
       (effects (font (size 1.27 1.27)) (justify left))
     )
-    (property "Footprint" "" (id 2) (at 101.6 115.57 0)
+    (property "Footprint" "" (id 2) (at 110.49 110.49 0)
       (effects (font (size 1.27 1.27)) hide)
     )
-    (property "Datasheet" "" (id 3) (at 101.6 115.57 0)
+    (property "Datasheet" "" (id 3) (at 110.49 110.49 0)
       (effects (font (size 1.27 1.27)) hide)
     )
     (pin "1")
   )
-  (symbol (lib_id "power:GND") (at 101.6 113.03 90) (unit 1)
+  (symbol (lib_id "power:GND") (at 110.49 113.03 90) (unit 1)
     (in_bom yes) (on_board yes) (fields_autoplaced)
-    (property "Reference" "#PWR01" (id 0) (at 107.95 113.03 0)
+    (property "Reference" "#PWR01" (id 0) (at 116.84 113.03 0)
       (effects (font (size 1.27 1.27)) hide)
     )
-    (property "Value" "GND" (id 1) (at 105.41 113.0299 90)
+    (property "Value" "GND" (id 1) (at 114.3 113.0299 90)
       (effects (font (size 1.27 1.27)) (justify right))
     )
-    (property "Footprint" "" (id 2) (at 101.6 113.03 0)
+    (property "Footprint" "" (id 2) (at 110.49 113.03 0)
       (effects (font (size 1.27 1.27)) hide)
     )
-    (property "Datasheet" "" (id 3) (at 101.6 113.03 0)
+    (property "Datasheet" "" (id 3) (at 110.49 113.03 0)
       (effects (font (size 1.27 1.27)) hide)
     )
     (pin "1")
   )
-  (symbol (lib_id "Connector:AudioJack3") (at 96.52 113.03 0) (unit 1)
+  (symbol (lib_id "Connector:AudioJack4") (at 105.41 113.03 0) (unit 1)
     (in_bom yes) (on_board yes) (fields_autoplaced)
-    (property "Reference" "J3" (id 0) (at 94.615 104.14 0))
-    (property "Value" "AudioJack3" (id 1) (at 94.615 106.68 0))
-    (property "Footprint" "Lily58:TRRS_JACK_MJ4PP9" (id 2) (at 96.52 113.03 0)
+    (property "Reference" "J3" (id 0) (at 119.38 118.11 0)
+      (effects (font (size 1.27 1.27)) (justify left))
+    )
+    (property "Value" "AudioJack3" (id 1) (at 109.22 120.65 0)
+      (effects (font (size 1.27 1.27)) (justify left))
+    )
+    (property "Footprint" "Keeb.io:TRRS-PJ-320A-Dual-Overlayed" (id 2) (at 105.41 106.68 0)
       (effects (font (size 1.27 1.27)) hide)
     )
-    (property "Datasheet" "~" (id 3) (at 96.52 113.03 0)
+    (property "Datasheet" "~" (id 3) (at 105.41 113.03 0)
       (effects (font (size 1.27 1.27)) hide)
     )
-    (pin "R")
-    (pin "S")
+    (pin "2")
+    (pin "3")
+    (pin "4")
     (pin "T")
   )
@@
     )
     (path "/a64269ba-b961-4619-8d5a-46f0ac7624d6"
-      (reference "J3") (unit 1) (value "AudioJack3") (footprint "Lily58:TRRS_JACK_MJ4PP9")
+      (reference "J3") (unit 1) (value "AudioJack3") (footprint "Keeb.io:TRRS-PJ-320A-Dual-Overlayed")
     )
     (path "/00000000-0000-0000-0000-0000613cdd8e"
@@
     )
     (path "/00000000-0000-0000-0000-00006300f927"
-      (reference "SWRST1") (unit 1) (value "SW_Push") (footprint "Keebio:SW_SPST_TL3342")
+      (reference "SWRST1") (unit 1) (value "SW_Push") (footprint "Keeb.io:SW_SPST_TL3342")
     )
     (path "/00000000-0000-0000-0000-0000613b76a4"
@@
     )
     (path "/00000000-0000-0000-0000-0000613bc179"
-      (reference "Y1") (unit 1) (value "16mhz") (footprint "Crystal:Resonator_SMD_muRata_CSTxExxV-3Pin_3.0x1.1mm_HandSoldering")
+      (reference "Y1") (unit 1) (value "16mhz") (footprint "Crystal:Resonator_SMD_Murata_CSTxExxV-3Pin_3.0x1.1mm")
     )
   )

Commit message: Changed USB-C port from Top-mount to Mid-mount
Parts:
- J1: footprint Connector_USB:USB_C_Receptacle_HRO_TYPE-C-31-M-12 -> Josh-Connectors:USB_C_TYPE-C-31-M-14
Changed lines of the file:
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@@
     (property "Reference" "J1" (id 0) (at 37.0078 99.8982 0))
     (property "Value" "Computer/Power" (id 1) (at 37.0078 102.2096 0))
-    (property "Footprint" "Connector_USB:USB_C_Receptacle_HRO_TYPE-C-31-M-12" (id 2) (at 38.1 121.92 0)
+    (property "Footprint" "Josh-Connectors:USB_C_TYPE-C-31-M-14" (id 2) (at 38.1 121.92 0)
       (effects (font (size 1.27 1.27)) hide)
     )
@@
     )
     (path "/00000000-0000-0000-0000-0000613c0548"
-      (reference "J1") (unit 1) (value "Computer/Power") (footprint "Connector_USB:USB_C_Receptacle_HRO_TYPE-C-31-M-12")
+      (reference "J1") (unit 1) (value "Computer/Power") (footprint "Josh-Connectors:USB_C_TYPE-C-31-M-14")
     )
     (path "/00000000-0000-0000-0000-000061403aef"
